File: HariFun_Stroboscope.sch (KiCad schematic (older format))
At the start: 7 parts

Commit message: Forgot to commit
Parts:
- gave numbers to parts that had none: 7
Other:
- moved on the sheet: D1, D2, D3, D4, Q1
Changed lines of the file:
@@
 $EndDescr
 $Comp
-L MCU_Module:Arduino_Nano_v3.x A?
+L MCU_Module:Arduino_Nano_v3.x A1
 U 1 1 5E6D06FA
 P 4900 3600
-F 0 "A?" H 4900 2511 50  0000 C CNN
+F 0 "A1" H 4900 2511 50  0000 C CNN
 F 1 "Arduino_Nano_v3.x" H 4900 2420 50  0000 C CNN
 F 2 "Module:Arduino_Nano" H 4900 3600 50  0001 C CIN
@@
 $EndComp
 $Comp
-L Device:R_POT RV?
+L Device:R_POT RV1
 U 1 1 5E6D1575
 P 3900 3600
-F 0 "RV?" H 3831 3646 50  0000 R CNN
+F 0 "RV1" H 3831 3646 50  0000 R CNN
 F 1 "10K" H 3831 3555 50  0000 R CNN
 F 2 "" H 3900 3600 50  0001 C CNN
@@
 $EndComp
 $Comp
-L power:+12V #PWR?
+L power:+12V #PWR02
 U 1 1 5E6D2834
-P 5900 2800
-F 0 "#PWR?" H 5900 2650 50  0001 C CNN
-F 1 "+12V" H 5915 2973 50  0000 C CNN
-F 2 "" H 5900 2800 50  0001 C CNN
-F 3 "" H 5900 2800 50  0001 C CNN
-	1    5900 2800
+P 6250 3400
+F 0 "#PWR02" H 6250 3250 50  0001 C CNN
+F 1 "+12V" H 6265 3573 50  0000 C CNN
+F 2 "" H 6250 3400 50  0001 C CNN
+F 3 "" H 6250 3400 50  0001 C CNN
+	1    6250 3400
 	1    0    0    -1
 $EndComp
 $Comp
-L Transistor_FET:IRLB8721PBF Q?
+L Transistor_FET:IRLB8721PBF Q1
 U 1 1 5E6D3080
-P 5800 4300
-F 0 "Q?" H 6004 4346 50  0000 L CNN
-F 1 "IRLB8721PBF" H 6004 4255 50  0000 L CNN
-F 2 "Package_TO_SOT_THT:TO-220-3_Vertical" H 6050 4225 50  0001 L CIN
-F 3 "http://www.infineon.com/dgdl/irlb8721pbf.pdf?fileId=5546d462533600a40153566056732591" H 5800 4300 50  0001 L CNN
-	1    5800 4300
+P 6150 4300
+F 0 "Q1" H 6354 4346 50  0000 L CNN
+F 1 "IRLB8721PBF" H 6354 4255 50  0000 L CNN
+F 2 "Package_TO_SOT_THT:TO-220-3_Vertical" H 6400 4225 50  0001 L CIN
+F 3 "http://www.infineon.com/dgdl/irlb8721pbf.pdf?fileId=5546d462533600a40153566056732591" H 6150 4300 50  0001 L CNN
+	1    6150 4300
 	1    0    0    -1
 $EndComp
 $Comp
-L power:GND #PWR?
+L power:GND #PWR01
 U 1 1 5E6D0E6C
 P 4900 5000
-F 0 "#PWR?" H 4900 4750 50  0001 C CNN
+F 0 "#PWR01" H 4900 4750 50  0001 C CNN
 F 1 "GND" H 4905 4827 50  0000 C CNN
 F 2 "" H 4900 5000 50  0001 C CNN
@@
 	4900 4900 4900 5000
 Wire Wire Line
-	4900 4900 5900 4900
-Wire Wire Line
-	5900 4900 5900 4500
-Wire Wire Line
 	3900 3750 3900 4900
 Wire Wire Line
@@
 	4050 3600 4400 3600
 Wire Wire Line
-	5400 4300 5600 4300
+	6050 3600 6250 3600
+Connection ~ 6250 3600
 Wire Wire Line
-	5700 3000 5900 3000
-Connection ~ 5900 3000
-Wire Wire Line
-	5900 3000 6050 3000
+	6250 3600 6400 3600
 $Comp
-L Device:LED D?
+L Device:LED D1
 U 1 1 5E6D2C37
-P 5700 3150
-F 0 "D?" V 5739 3033 50  0000 R CNN
-F 1 "LED" V 5648 3033 50  0000 R CNN
-F 2 "" H 5700 3150 50  0001 C CNN
-F 3 "~" H 5700 3150 50  0001 C CNN
-	1    5700 3150
+P 6050 3750
+F 0 "D1" V 6089 3633 50  0000 R CNN
+F 1 "LED" V 5998 3633 50  0000 R CNN
+F 2 "" H 6050 3750 50  0001 C CNN
+F 3 "~" H 6050 3750 50  0001 C CNN
+	1    6050 3750
 	0    -1   -1   0
 $EndComp
 $Comp
-L Device:LED D?
+L Device:LED D2
 U 1 1 5E6D3BFC
-P 6050 3150
-F 0 "D?" V 6089 3033 50  0000 R CNN
-F 1 "LED" V 5998 3033 50  0000 R CNN
-F 2 "" H 6050 3150 50  0001 C CNN
-F 3 "~" H 6050 3150 50  0001 C CNN
-	1    6050 3150
+P 6400 3750
+F 0 "D2" V 6439 3633 50  0000 R CNN
+F 1 "LED" V 6348 3633 50  0000 R CNN
+F 2 "" H 6400 3750 50  0001 C CNN
+F 3 "~" H 6400 3750 50  0001 C CNN
+	1    6400 3750
 	0    -1   -1   0
 $EndComp
-Connection ~ 6050 3000
+Connection ~ 6400 3600
 Wire Wire Line
-	6050 3000 6450 3000
+	6400 3600 6800 3600
 $Comp
-L Device:LED D?
+L Device:LED D3
 U 1 1 5E6D41C0
-P 6450 3150
-F 0 "D?" V 6489 3033 50  0000 R CNN
-F 1 "LED" V 6398 3033 50  0000 R CNN
-F 2 "" H 6450 3150 50  0001 C CNN
-F 3 "~" H 6450 3150 50  0001 C CNN
-	1    6450 3150
+P 6800 3750
+F 0 "D3" V 6839 3633 50  0000 R CNN
+F 1 "LED" V 6748 3633 50  0000 R CNN
+F 2 "" H 6800 3750 50  0001 C CNN
+F 3 "~" H 6800 3750 50  0001 C CNN
+	1    6800 3750
 	0    -1   -1   0
 $EndComp
-Connection ~ 6450 3000
+Connection ~ 6800 3600
 $Comp
-L Device:LED D?
+L Device:LED D4
 U 1 1 5E6D4465
-P 6850 3150
-F 0 "D?" V 6889 3033 50  0000 R CNN
-F 1 "LED" V 6798 3033 50  0000 R CNN
-F 2 "" H 6850 3150 50  0001 C CNN
-F 3 "~" H 6850 3150 50  0001 C CNN
-	1    6850 3150
+P 7200 3750
+F 0 "D4" V 7239 3633 50  0000 R CNN
+F 1 "LED" V 7148 3633 50  0000 R CNN
+F 2 "" H 7200 3750 50  0001 C CNN
+F 3 "~" H 7200 3750 50  0001 C CNN
+	1    7200 3750
 	0    -1   -1   0
 $EndComp
 Wire Wire Line
-	6450 3000 6850 3000
+	6800 3600 7200 3600
 Wire Wire Line
-	6850 3000 7450 3000
-Connection ~ 6850 3000
+	7200 3600 7800 3600
+Connection ~ 7200 3600
 Wire Wire Line
-	5700 3300 5900 3300
-Connection ~ 6050 3300
+	6050 3900 6250 3900
+Connection ~ 6400 3900
 Wire Wire Line
-	6050 3300 6450 3300
-Connection ~ 6450 3300
+	6400 3900 6800 3900
+Connection ~ 6800 3900
 Wire Wire Line
-	6450 3300 6850 3300
-Connection ~ 6850 3300
+	6800 3900 7200 3900
+Connection ~ 7200 3900
 Wire Wire Line
-	6850 3300 7450 3300
-Connection ~ 5900 3300
+	7200 3900 7800 3900
+Connection ~ 6250 3900
 Wire Wire Line
-	5900 3300 6050 3300
+	6250 3900 6400 3900
 Wire Wire Line
-	5900 3300 5900 4100
+	6250 3900 6250 4100
 Text Notes 4400 2400 0    50   ~ 0
 Arduino is powered by USB port
-Text Notes 6050 2800 0    50   ~ 0
+Text Notes 6350 3450 0    50   ~ 0
 LEDs are powered separately
 Wire Wire Line
@@
 	4700 2500 4700 2600
 Wire Wire Line
-	5900 2800 5900 3000
+	6250 3400 6250 3600
+Wire Wire Line
+	6250 4500 6250 4900
+Wire Wire Line
+	5400 4300 5950 4300
+Wire Wire Line
+	4900 4900 6250 4900
 $EndSCHEMATC
